Commit message: First working version of Maxon motor working in sim

File: embr_sim/ros2_ws/src/embr_description/urdf/maxon_motor/urdf/maxon_motor.urdf.xacro (robot description, xacro)
@@ -10,5 +10,5 @@
             <origin xyz="0 0 0" rpy="0 -0 0" />
             <geometry>
-                <mesh filename="package://maxon_motor/meshes/Body.stl" scale="1 1 1" />
+                <mesh filename="package://embr_description/meshes/maxon_motor/meshes/Body.stl" scale="1 1 1" />
             </geometry>
             <material name="0.501961_0.501961_0.501961_0.000000_0.000000">
@@ -27,5 +27,5 @@
             <origin xyz="0 0.0204 -9.093e-19" rpy="0 -0 0" />
             <geometry>
-                <mesh filename="package://maxon_motor/meshes/Shaft.stl" scale="1 1 1" />
+                <mesh filename="package://embr_description/meshes/maxon_motor/meshes/Shaft.stl" scale="1 1 1" />
             </geometry>
             <material name="0.901961_0.901961_0.901961_0.000000_0.000000">
@@ -43,5 +43,5 @@
             <origin xyz="8.67362e-19 -0.0133 3.18908e-19" rpy="0 -0 0" />
             <geometry>
-                <mesh filename="package://maxon_motor/meshes/Tab_1.stl" scale="1 1 1" />
+                <mesh filename="package://embr_description/meshes/maxon_motor/meshes/Tab_1.stl" scale="1 1 1" />
             </geometry>
             <material name="0.917647_0.917647_0.917647_0.000000_0.000000">
@@ -59,5 +59,5 @@
             <origin xyz="-8.67362e-19 -0.0133 3.08814e-19" rpy="0 -0 0" />
             <geometry>
-                <mesh filename="package://maxon_motor/meshes/Tab_2.stl" scale="1 1 1" />
+                <mesh filename="package://embr_description/meshes/maxon_motor/meshes/Tab_2.stl" scale="1 1 1" />
             </geometry>
             <material name="0.917647_0.917647_0.917647_0.000000_0.000000">
