Commit message: Teleop Twist Component working and proof of concept with rviz2 responding to commands

File: embr_phys/ros2_ws/src/embr_description/urdf/embr_simple/urdf/embr_simple.urdf (robot description, URDF)
Before this commit: robot embr_simple, 22 links, 21 joints
Links:
- removed link maxon_body
- removed link maxon_body_1
- removed link maxon_body_2
- removed link maxon_body_3
- removed link maxon_shaft
- removed link maxon_shaft_1
- removed link maxon_shaft_2
- removed link maxon_shaft_3
- removed link maxon_tab_left
- removed link maxon_tab_left_1
- removed link maxon_tab_left_2
- removed link maxon_tab_left_3
- removed link maxon_tab_right
- removed link maxon_tab_right_1
- removed link maxon_tab_right_2
- removed link maxon_tab_right_3
- removed link wheel
- removed link wheel_1
- removed link wheel_2
- removed link wheel_3
Joints:
- removed joint shaft_dof
- removed joint shaft_dof_1
- removed joint shaft_dof_2
- removed joint shaft_dof_3
- removed joint wheel_shaft
- removed joint wheel_shaft_1
- removed joint wheel_shaft_2
- removed joint wheel_shaft_3
- added joint front_left_maxon: type continuous, parent maxon_body_1, child maxon_front_left_shaft, origin xyz=-2.77556e-17 ${-motor_shaft_offset} 1.11022e-16 rpy=-3.14159 1.52785 5.45973e-15, axis 0 1 0
- added joint front_right_maxon: type continuous, parent maxon_body, child maxon_front_right_shaft, origin xyz=-1.38778e-17 ${-motor_shaft_offset} 0 rpy=0 1.5708 3.14159, axis 0 1 0
- added joint rear_left_maxon: type continuous, parent maxon_body_2, child maxon_rear_left_shaft, origin xyz=0 ${-motor_shaft_offset} 4.16334e-17 rpy=3.14159 1.52785 -4.69359e-15, axis 0 1 0
- added joint rear_right_maxon: type continuous, parent maxon_body_3, child maxon_rear_right_shaft, origin xyz=-2.77556e-17 ${-motor_shaft_offset} -1.38778e-17 rpy=0 1.5708 3.14159, axis 0 1 0
- added joint shaft_front_left_wheel: type fixed, parent maxon_front_left_shaft, child wheel_front_left, origin xyz=5.55112e-17 ${wheel_mount_offset} -1.38778e-17 rpy=3.0271e-19 0.23032 -3.14159, axis 0 -1 0
- added joint shaft_front_right_wheel: type fixed, parent maxon_front_right_shaft, child wheel_front_right, origin xyz=5.55112e-17 ${wheel_mount_offset} -1.38778e-17 rpy=-2.89829e-20 0.23032 3.14159, axis 0 -1 0
- added joint shaft_rear_left_wheel: type fixed, parent maxon_rear_left_shaft, child wheel_rear_left, origin xyz=0 ${wheel_mount_offset} 1.38778e-17 rpy=-2.2294e-18 0.23032 3.14159, axis 0 -1 0
- added joint shaft_rear_right_wheel: type fixed, parent maxon_rear_right_shaft, child wheel_rear_right, origin xyz=-1.38778e-17 ${wheel_mount_offset} 0 rpy=-9.24232e-19 0.23032 3.14159, axis 0 -1 0
- joint fastened_1: origin xyz=-0.0225927 0.0867344 0.0122 rpy=0 -1.5708 -1.5708 -> xyz=${motor_mount_center_x - motor_mount_half_span} ${wheelbase / 2} ${motor_mount_height} rpy=0 -1.5708 -1.5708
- joint fastened_2: origin xyz=0.0267554 0.0867344 0.0122 rpy=0 -1.5708 1.5708 -> xyz=${motor_mount_center_x + motor_mount_half_span} ${wheelbase / 2} ${motor_mount_height} rpy=0 -1.5708 1.5708
- joint fastened_3: origin xyz=0.0267554 -0.0867344 0.0122 rpy=0 -1.5708 1.5708 -> xyz=${motor_mount_center_x + motor_mount_half_span} ${-wheelbase / 2} ${motor_mount_height} rpy=0 -1.5708 1.5708
- joint fastened_4: origin xyz=-0.0225927 -0.0867344 0.0122 rpy=0 -1.5708 -1.5708 -> xyz=${motor_mount_center_x - motor_mount_half_span} ${-wheelbase / 2} ${motor_mount_height} rpy=0 -1.5708 -1.5708
- joint fixed_node_to_root_joint: origin xyz=-0.0521915 0.198476 -0.0944215 rpy=-0.0211084 0.0124172 -3.11206 -> xyz=0 0 0 rpy=0 0 ${pi / 2}
- joint left_tab_fastener: origin xyz=-0.005 0 1.11022e-16 rpy=3.55889e-16 -3.90486e-15 -1.7434e-16 -> xyz=${-tab_mount_offset} 0 1.11022e-16 rpy=3.55889e-16 -3.90486e-15 -1.7434e-16
- joint left_tab_fastener_1: origin xyz=-0.005 -6.93889e-18 -5.55112e-17 rpy=5.47522e-16 2.1684e-16 1.13624e-16 -> xyz=${-tab_mount_offset} -6.93889e-18 -5.55112e-17 rpy=5.47522e-16 2.1684e-16 1.13624e-16
- joint left_tab_fastener_2: origin xyz=-0.005 -1.38778e-17 4.16334e-17 rpy=-1.23274e-16 1.43982e-16 -7.97973e-17 -> xyz=${-tab_mount_offset} -1.38778e-17 4.16334e-17 rpy=-1.23274e-16 1.43982e-16 -7.97973e-17
- joint left_tab_fastener_3: origin xyz=-0.005 -8.32667e-17 -1.38778e-17 rpy=1.11708e-15 -1.03043e-15 -6.245e-16 -> xyz=${-tab_mount_offset} -8.32667e-17 -1.38778e-17 rpy=1.11708e-15 -1.03043e-15 -6.245e-16
- joint right_tab_fastener: origin xyz=0.005 4.16334e-17 0 rpy=3.55889e-16 -3.90486e-15 -1.7434e-16 -> xyz=${tab_mount_offset} 4.16334e-17 0 rpy=3.55889e-16 -3.90486e-15 -1.7434e-16
- joint right_tab_fastener_1: origin xyz=0.005 -6.93889e-18 -1.11022e-16 rpy=5.47522e-16 2.1684e-16 1.13624e-16 -> xyz=${tab_mount_offset} -6.93889e-18 -1.11022e-16 rpy=5.47522e-16 2.1684e-16 1.13624e-16
- joint right_tab_fastener_2: origin xyz=0.005 0 4.16334e-17 rpy=-1.23274e-16 1.43982e-16 -7.97973e-17 -> xyz=${tab_mount_offset} 0 4.16334e-17 rpy=-1.23274e-16 1.43982e-16 -7.97973e-17
- joint right_tab_fastener_3: origin xyz=0.005 -1.04083e-16 -1.38778e-17 rpy=1.11708e-15 -1.03043e-15 -6.245e-16 -> xyz=${tab_mount_offset} -1.04083e-16 -1.38778e-17 rpy=1.11708e-15 -1.03043e-15 -6.245e-16
